Commit message: refined once

File: swarm_robotics_urdf/src/urdf/swarm1.xacro (robot description, xacro)
@@ -14,5 +14,5 @@
     <xacro:property name="bodyOX" value="0" />
     <xacro:property name="bodyOY" value="0" />
-    <xacro:property name="bodyOZ" value="0.0127" />
+    <xacro:property name="bodyOZ" value="0.01" />
     <!-- define the drive-wheel dimensions-->
     <xacro:property name="tirediam" value="0.03" />
@@ -69,5 +69,5 @@
   <inertial>
     <mass value="0.3" />
-    <origin xyz="0 0 0.0127" />
+    <origin xyz="0 0 ${bodyOZ}" />
     <inertia ixx="0.032258" ixy="0.0" ixz="0.0"
       iyy="20.2258" iyz="0.0"
@@ -96,11 +96,11 @@
  </gazebo>
   <gazebo reference="right_wheel">
-    <mu1>1000</mu1>
-    <mu2>1000</mu2>
+    <mu1>100000</mu1>
+    <mu2>100000</mu2>
     <material>Gazebo/Green</material>
   </gazebo>
   <gazebo reference="left_wheel">
-    <mu1>1000</mu1>
-    <mu2>1000</mu2>
+    <mu1>100000</mu1>
+    <mu2>100000</mu2>
     <material>Gazebo/Red</material>
   </gazebo>
@@ -122,5 +122,5 @@
       </visual>
       <inertial>
-          <mass value="0.000001" />
+          <mass value="0.00000001" />
           <origin xyz="0 0 0" rpy="0 0 0"/>
           <inertia ixx="0.000032258" ixy="0" ixz="0" iyy="0.000032258" iyz="0" izz="0.000032258" />
@@ -129,5 +129,5 @@
   <joint name="lidar_joint" type="fixed">
       <axis xyz="0 1 0" />
-      <origin xyz="${bodyOX} ${bodyOY} ${tirerad}" rpy="0 0 0"/>
+      <origin xyz="${bodyOX} ${bodyOY} ${bodyheight}" rpy="0 0 0"/>
       <parent link="base_link"/>
       <child link="lidar_link"/>

File: swarm_robotics_urdf/src/urdf/swarm2.xacro (robot description, xacro)
@@ -14,5 +14,5 @@
     <xacro:property name="bodyOX" value="0" />
     <xacro:property name="bodyOY" value="0" />
-    <xacro:property name="bodyOZ" value="0.0127" />
+    <xacro:property name="bodyOZ" value="0.01" />
     <!-- define the drive-wheel dimensions-->
     <xacro:property name="tirediam" value="0.03" />
@@ -69,5 +69,5 @@
   <inertial>
     <mass value="0.3" />
-    <origin xyz="0 0 0.0127" />
+    <origin xyz="0 0 ${bodyOZ}" />
     <inertia ixx="0.032258" ixy="0.0" ixz="0.0"
       iyy="20.2258" iyz="0.0"
@@ -96,11 +96,11 @@
  </gazebo>
   <gazebo reference="right_wheel">
-    <mu1>1000</mu1>
-    <mu2>1000</mu2>
+    <mu1>100000</mu1>
+    <mu2>100000</mu2>
     <material>Gazebo/Green</material>
   </gazebo>
   <gazebo reference="left_wheel">
-    <mu1>1000</mu1>
-    <mu2>1000</mu2>
+    <mu1>100000</mu1>
+    <mu2>100000</mu2>
     <material>Gazebo/Red</material>
   </gazebo>
@@ -122,5 +122,5 @@
       </visual>
       <inertial>
-          <mass value="0.000001" />
+          <mass value="0.00000001" />
           <origin xyz="0 0 0" rpy="0 0 0"/>
           <inertia ixx="0.000032258" ixy="0" ixz="0" iyy="0.000032258" iyz="0" izz="0.000032258" />
@@ -129,5 +129,5 @@
   <joint name="lidar_joint" type="fixed">
       <axis xyz="0 1 0" />
-      <origin xyz="${bodyOX} ${bodyOY} ${tirerad}" rpy="0 0 0"/>
+      <origin xyz="${bodyOX} ${bodyOY} ${bodyOZ}" rpy="0 0 0"/>
       <parent link="base_link"/>
       <child link="lidar_link"/>

File: swarm_robotics_urdf/src/urdf/swarm3.xacro (robot description, xacro)
@@ -14,5 +14,5 @@
     <xacro:property name="bodyOX" value="0" />
     <xacro:property name="bodyOY" value="0" />
-    <xacro:property name="bodyOZ" value="0.0127" />
+    <xacro:property name="bodyOZ" value="0.01" />
     <!-- define the drive-wheel dimensions-->
     <xacro:property name="tirediam" value="0.03" />
@@ -69,5 +69,5 @@
   <inertial>
     <mass value="0.3" />
-    <origin xyz="0 0 0.0127" />
+    <origin xyz="0 0 ${bodyOZ}" />
     <inertia ixx="0.032258" ixy="0.0" ixz="0.0"
       iyy="20.2258" iyz="0.0"
@@ -96,11 +96,11 @@
  </gazebo>
   <gazebo reference="right_wheel">
-    <mu1>1000</mu1>
-    <mu2>1000</mu2>
+    <mu1>100000</mu1>
+    <mu2>100000</mu2>
     <material>Gazebo/Green</material>
   </gazebo>
   <gazebo reference="left_wheel">
-    <mu1>1000</mu1>
-    <mu2>1000</mu2>
+    <mu1>100000</mu1>
+    <mu2>100000</mu2>
     <material>Gazebo/Red</material>
   </gazebo>
@@ -122,5 +122,5 @@
       </visual>
       <inertial>
-          <mass value="0.000001" />
+          <mass value="0.00000001" />
           <origin xyz="0 0 0" rpy="0 0 0"/>
           <inertia ixx="0.000032258" ixy="0" ixz="0" iyy="0.000032258" iyz="0" izz="0.000032258" />
@@ -129,5 +129,5 @@
   <joint name="lidar_joint" type="fixed">
       <axis xyz="0 1 0" />
-      <origin xyz="${bodyOX} ${bodyOY} ${tirerad}" rpy="0 0 0"/>
+      <origin xyz="${bodyOX} ${bodyOY} ${bodyOZ}" rpy="0 0 0"/>
       <parent link="base_link"/>
       <child link="lidar_link"/>

File: swarm_robotics_urdf/src/urdf/swarm4.xacro (robot description, xacro)
@@ -14,5 +14,5 @@
     <xacro:property name="bodyOX" value="0" />
     <xacro:property name="bodyOY" value="0" />
-    <xacro:property name="bodyOZ" value="0.0127" />
+    <xacro:property name="bodyOZ" value="0.01" />
     <!-- define the drive-wheel dimensions-->
     <xacro:property name="tirediam" value="0.03" />
@@ -69,5 +69,5 @@
   <inertial>
     <mass value="0.3" />
-    <origin xyz="0 0 0.0127" />
+    <origin xyz="0 0 ${bodyOZ}" />
     <inertia ixx="0.032258" ixy="0.0" ixz="0.0"
       iyy="20.2258" iyz="0.0"
@@ -96,11 +96,11 @@
  </gazebo>
   <gazebo reference="right_wheel">
-    <mu1>1000</mu1>
-    <mu2>1000</mu2>
+    <mu1>100000</mu1>
+    <mu2>100000</mu2>
     <material>Gazebo/Green</material>
   </gazebo>
   <gazebo reference="left_wheel">
-    <mu1>1000</mu1>
-    <mu2>1000</mu2>
+    <mu1>100000</mu1>
+    <mu2>100000</mu2>
     <material>Gazebo/Red</material>
   </gazebo>
@@ -129,5 +129,5 @@
   <joint name="lidar_joint" type="fixed">
       <axis xyz="0 1 0" />
-      <origin xyz="${bodyOX} ${bodyOY} ${tirerad}" rpy="0 0 0"/>
+      <origin xyz="${bodyOX} ${bodyOY} ${bodyOZ}" rpy="0 0 0"/>
       <parent link="base_link"/>
       <child link="lidar_link"/>

File: swarm_robotics_urdf/src/urdf/swarm5.xacro (robot description, xacro)
@@ -14,5 +14,5 @@
     <xacro:property name="bodyOX" value="0" />
     <xacro:property name="bodyOY" value="0" />
-    <xacro:property name="bodyOZ" value="0.0127" />
+    <xacro:property name="bodyOZ" value="0.01" />
     <!-- define the drive-wheel dimensions-->
     <xacro:property name="tirediam" value="0.03" />
@@ -69,5 +69,5 @@
   <inertial>
     <mass value="0.3" />
-    <origin xyz="0 0 0.0127" />
+    <origin xyz="0 0 ${bodyOZ}" />
     <inertia ixx="0.032258" ixy="0.0" ixz="0.0"
       iyy="20.2258" iyz="0.0"
@@ -96,11 +96,11 @@
  </gazebo>
   <gazebo reference="right_wheel">
-    <mu1>1000</mu1>
-    <mu2>1000</mu2>
+    <mu1>100000</mu1>
+    <mu2>100000</mu2>
     <material>Gazebo/Green</material>
   </gazebo>
   <gazebo reference="left_wheel">
-    <mu1>1000</mu1>
-    <mu2>1000</mu2>
+    <mu1>100000</mu1>
+    <mu2>100000</mu2>
     <material>Gazebo/Red</material>
   </gazebo>
@@ -129,5 +129,5 @@
   <joint name="lidar_joint" type="fixed">
       <axis xyz="0 1 0" />
-      <origin xyz="${bodyOX} ${bodyOY} ${tirerad}" rpy="0 0 0"/>
+      <origin xyz="${bodyOX} ${bodyOY} ${bodyOZ}" rpy="0 0 0"/>
       <parent link="base_link"/>
       <child link="lidar_link"/>

File: swarm_robotics_urdf/src/urdf/swarm6.xacro (robot description, xacro)
@@ -14,5 +14,5 @@
     <xacro:property name="bodyOX" value="0" />
     <xacro:property name="bodyOY" value="0" />
-    <xacro:property name="bodyOZ" value="0.0127" />
+    <xacro:property name="bodyOZ" value="0.01" />
     <!-- define the drive-wheel dimensions-->
     <xacro:property name="tirediam" value="0.03" />
@@ -69,5 +69,5 @@
   <inertial>
     <mass value="0.3" />
-    <origin xyz="0 0 0.0127" />
+    <origin xyz="0 0 ${bodyOZ}" />
     <inertia ixx="0.032258" ixy="0.0" ixz="0.0"
       iyy="20.2258" iyz="0.0"
@@ -96,11 +96,11 @@
  </gazebo>
   <gazebo reference="right_wheel">
-    <mu1>1000</mu1>
-    <mu2>1000</mu2>
+    <mu1>100000</mu1>
+    <mu2>100000</mu2>
     <material>Gazebo/Green</material>
   </gazebo>
   <gazebo reference="left_wheel">
-    <mu1>1000</mu1>
-    <mu2>1000</mu2>
+    <mu1>100000</mu1>
+    <mu2>100000</mu2>
     <material>Gazebo/Red</material>
   </gazebo>
@@ -129,5 +129,5 @@
   <joint name="lidar_joint" type="fixed">
       <axis xyz="0 1 0" />
-      <origin xyz="${bodyOX} ${bodyOY} ${tirerad}" rpy="0 0 0"/>
+      <origin xyz="${bodyOX} ${bodyOY} ${bodyOZ}" rpy="0 0 0"/>
       <parent link="base_link"/>
       <child link="lidar_link"/>

File: swarm_robotics_urdf/src/urdf/test_try.xacro (robot description, xacro)
@@ -14,5 +14,5 @@
     <xacro:property name="bodyOX" value="0" />
     <xacro:property name="bodyOY" value="0" />
-    <xacro:property name="bodyOZ" value="0.0127" />
+    <xacro:property name="bodyOZ" value="0.0100" />
     <!-- define the drive-wheel dimensions-->
     <xacro:property name="tirediam" value="0.03" />
@@ -69,5 +69,5 @@
   <inertial>
     <mass value="0.3" />
-    <origin xyz="0 0 0.0127" />
+    <origin xyz="0 0 ${bodyOZ}" />
     <inertia ixx="0.032258" ixy="0.0" ixz="0.0"
       iyy="20.2258" iyz="0.0"
@@ -96,11 +96,11 @@
  </gazebo>
   <gazebo reference="right_wheel">
-    <mu1>1000</mu1>
-    <mu2>1000</mu2>
+    <mu1>100000</mu1>
+    <mu2>100000</mu2>
     <material>Gazebo/Green</material>
   </gazebo>
   <gazebo reference="left_wheel">
-    <mu1>1000</mu1>
-    <mu2>1000</mu2>
+    <mu1>100000</mu1>
+    <mu2>100000</mu2>
     <material>Gazebo/Red</material>
   </gazebo>
@@ -122,5 +122,5 @@
       </visual>
       <inertial>
-          <mass value="0.000001" />
+          <mass value="0.00000001" />
           <origin xyz="0 0 0" rpy="0 0 0"/>
           <inertia ixx="0.000032258" ixy="0" ixz="0" iyy="0.000032258" iyz="0" izz="0.000032258" />
@@ -129,5 +129,5 @@
   <joint name="lidar_joint" type="fixed">
       <axis xyz="0 1 0" />
-      <origin xyz="${bodyOX} ${bodyOY} ${tirerad}" rpy="0 0 0"/>
+      <origin xyz="${bodyOX} ${bodyOY} ${bodyheight}" rpy="0 0 0"/>
       <parent link="base_link"/>
       <child link="lidar_link"/>
