Commit message: add sensing fusions and angles

File: urdf/iRobot1.urdf (robot description, URDF)
Before this commit: robot iRobot, 11 links, 10 joints
Joints:
- joint hokuyo_laser_joint: origin xyz=0 0 0.06 rpy=0 0 0 -> xyz=0 0 0.1 rpy=0 0 0

File: urdf/iRobot2.urdf (robot description, URDF)
Before this commit: robot iRobot, 11 links, 10 joints
Joints:
- joint hokuyo_laser_joint: origin xyz=0 0 0.06 rpy=0 0 0 -> xyz=0 0 0.1 rpy=0 0 0

File: urdf/iRobot3.urdf (robot description, URDF)
Before this commit: robot iRobot, 11 links, 10 joints
Joints:
- joint hokuyo_laser_joint: origin xyz=0 0 0.06 rpy=0 0 0 -> xyz=0 0 0.1 rpy=0 0 0
